Commit message: Fix meshes not found

File: description_files/urdf/g1_23dof.urdf (robot description, URDF)
Before this commit: robot g1_23dof_rev_1_0, 48 links, 47 joints
Links:
- link head_link: geometry collision mesh filename=package://hurobots/description_files/meshes/head_link.STL; visual mesh filename=package://hurobots/description_files/meshes/head_link.STL
- link left_ankle_pitch_link: geometry collision mesh filename=package://hurobots/description_files/meshes/left_ankle_pitc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; visual mesh filename=package://hurobots/description_files/meshes/left_ankle_pitc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
- link left_ankle_roll_link: geometry collision sphere radius=0.005; collision sphere radius=0.005
- link left_elbow_link: geometry collision mesh filename=package://hurobots/description_files/meshes/left_elbow_link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; visual mesh filename=package://hurobots/description_files/meshes/left_elbow_link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
- link left_hip_pitch_link: geometry collision mesh filename=package://hurobots/description_files/meshes/left_hip_pitch_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; visual mesh filename=package://hurobots/description_files/meshes/left_hip_pitch_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
- link left_hip_roll_link: geometry collision mesh filename=package://hurobots/description_files/meshes/left_hip_roll_l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; visual mesh filename=package://hurobots/description_files/meshes/left_hip_roll_l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
- link left_hip_yaw_link: geometry collision mesh filename=package://hurobots/description_files/meshes/left_hip_yaw_li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; visual mesh filename=package://hurobots/description_files/meshes/left_hip_yaw_li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
- link left_knee_link: geometry collision mesh filename=package://hurobots/description_files/meshes/left_knee_link.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; visual mesh filename=package://hurobots/description_files/meshes/left_knee_link.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
- link left_shoulder_pitch_link: geometry collision cylinder length=0.05 radius=0.03; visual mesh filename=package://hurobots/description_files/meshes/left_shoulder_p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
- link left_shoulder_roll_link: geometry collision cylinder length=0.03 radius=0.03; visual mesh filename=package://hurobots/description_files/meshes/left_shoulder_r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
- link left_shoulder_yaw_link: geometry collision mesh filename=package://hurobots/description_files/meshes/left_shoulder_y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; visual mesh filename=package://hurobots/description_files/meshes/left_shoulder_y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
- link left_wrist_roll_rubber_hand: geometry collision mesh filename=package://hurobots/description_files/meshes/left_wrist_roll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; visual mesh filename=package://hurobots/description_files/meshes/left_wrist_roll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
- link logo_link: geometry collision mesh filename=package://hurobots/description_files/meshes/logo_link.STL; visual mesh filename=package://hurobots/description_files/meshes/logo_link.STL
- link pelvis: geometry visual mesh filename=package://hurobots/description_files/meshes/pelvis.STL
- link pelvis_contour_link: geometry collision mesh filename=package://hurobots/description_files/meshes/pelvis_contour_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; visual mesh filename=package://hurobots/description_files/meshes/pelvis_contour_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
- link right_ankle_pitch_link: geometry collision mesh filename=package://hurobots/description_files/meshes/right_ankle_pit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; visual mesh filename=package://hurobots/description_files/meshes/right_ankle_pit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
- link right_ankle_roll_link: geometry collision sphere radius=0.005; collision sphere radius=0.005
- link right_elbow_link: geometry collision mesh filename=package://hurobots/description_files/meshes/right_elbow_lin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; visual mesh filename=package://hurobots/description_files/meshes/right_elbow_lin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
- link right_hip_pitch_link: geometry collision mesh filename=package://hurobots/description_files/meshes/right_hip_pitch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; visual mesh filename=package://hurobots/description_files/meshes/right_hip_pitch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
- link right_hip_roll_link: geometry collision mesh filename=package://hurobots/description_files/meshes/right_hip_roll_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; visual mesh filename=package://hurobots/description_files/meshes/right_hip_roll_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
- link right_hip_yaw_link: geometry collision mesh filename=package://hurobots/description_files/meshes/right_hip_yaw_l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; visual mesh filename=package://hurobots/description_files/meshes/right_hip_yaw_l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
- link right_knee_link: geometry collision mesh filename=package://hurobots/description_files/meshes/right_knee_link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; visual mesh filename=package://hurobots/description_files/meshes/right_knee_link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
- link right_shoulder_pitch_link: geometry collision cylinder length=0.05 radius=0.03; visual mesh filename=package://hurobots/description_files/meshes/right_shoulder_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
- link right_shoulder_roll_link: geometry collision cylinder length=0.03 radius=0.03; visual mesh filename=package://hurobots/description_files/meshes/right_shoulder_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
- link right_shoulder_yaw_link: geometry collision mesh filename=package://hurobots/description_files/meshes/right_shoulder_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; visual mesh filename=package://hurobots/description_files/meshes/right_shoulder_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
- link right_wrist_roll_rubber_hand: geometry collision mesh filename=package://hurobots/description_files/meshes/right_wrist_rol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; visual mesh filename=package://hurobots/description_files/meshes/right_wrist_rol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
- link torso_link: geometry collision mesh filename=package://hurobots/description_files/meshes/torso_link_23do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; visual mesh filename=package://hurobots/description_files/meshes/torso_link_23do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

File: description_files/urdf/g1_23dof_rubber_hands.urdf (robot description, URDF)
Before this commit: robot g1_23dof_rubber_hands, 31 links, 30 joints
Links:
- link head_link: geometry visual mesh filename=package://hurobots/description_files/meshes/head_link.STL
- link left_ankle_pitch_link: geometry visual mesh filename=package://hurobots/description_files/meshes/left_ankle_pitc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
- link left_ankle_roll_link: geometry collision box size=0.20311 0.0647 0.01851; visual mesh filename=package://hurobots/description_files/meshes/left_ankle_roll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
- link left_elbow_link: geometry visual mesh filename=package://hurobots/description_files/meshes/left_elbow_link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
- link left_hip_pitch_link: geometry visual mesh filename=package://hurobots/description_files/meshes/left_hip_pitch_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
- link left_hip_roll_link: geometry visual mesh filename=package://hurobots/description_files/meshes/left_hip_roll_l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
- link left_hip_yaw_link: geometry visual mesh filename=package://hurobots/description_files/meshes/left_hip_yaw_li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
- link left_knee_link: geometry visual mesh filename=package://hurobots/description_files/meshes/left_knee_link.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
- link left_shoulder_pitch_link: geometry visual mesh filename=package://hurobots/description_files/meshes/left_shoulder_p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
- link left_shoulder_roll_link: geometry visual mesh filename=package://hurobots/description_files/meshes/left_shoulder_r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
- link left_shoulder_yaw_link: geometry collision sphere radius=0.04; visual mesh filename=package://hurobots/description_files/meshes/left_shoulder_y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
- link left_wrist_roll_rubber_hand: geometry collision mesh filename=package://hurobots/description_files/meshes/left_wrist_roll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; visual mesh filename=package://hurobots/description_files/meshes/left_wrist_roll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
- link logo_link: geometry visual mesh filename=package://hurobots/description_files/meshes/logo_link.STL
- link pelvis: geometry visual mesh filename=package://hurobots/description_files/meshes/pelvis.STL
- link pelvis_contour_link: geometry visual mesh filename=package://hurobots/description_files/meshes/pelvis_contour_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
- link right_ankle_pitch_link: geometry visual mesh filename=package://hurobots/description_files/meshes/right_ankle_pit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
- link right_ankle_roll_link: geometry collision box size=0.20311 0.0647 0.01851; visual mesh filename=package://hurobots/description_files/meshes/right_ankle_rol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
- link right_elbow_link: geometry visual mesh filename=package://hurobots/description_files/meshes/right_elbow_lin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
- link right_hip_pitch_link: geometry visual mesh filename=package://hurobots/description_files/meshes/right_hip_pitch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
- link right_hip_roll_link: geometry visual mesh filename=package://hurobots/description_files/meshes/right_hip_roll_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
- link right_hip_yaw_link: geometry visual mesh filename=package://hurobots/description_files/meshes/right_hip_yaw_l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
- link right_knee_link: geometry visual mesh filename=package://hurobots/description_files/meshes/right_knee_link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
- link right_shoulder_pitch_link: geometry visual mesh filename=package://hurobots/description_files/meshes/right_shoulder_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
- link right_shoulder_roll_link: geometry visual mesh filename=package://hurobots/description_files/meshes/right_shoulder_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
- link right_shoulder_yaw_link: geometry collision sphere radius=0.04; visual mesh filename=package://hurobots/description_files/meshes/right_shoulder_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
- link right_wrist_roll_rubber_hand: geometry collision mesh filename=package://hurobots/description_files/meshes/right_wrist_rol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; visual mesh filename=package://hurobots/description_files/meshes/right_wrist_rol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
- link torso_link: geometry collision mesh filename=package://hurobots/description_files/meshes/torso_link_23do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; visual mesh filename=package://hurobots/description_files/meshes/torso_link_23do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

File: description_files/urdf/g1_23dof_rubber_hands_foot_collisions.urdf (robot description, URDF)
Before this commit: robot g1_23dof_rubber_hands, 39 links, 38 joints
Links:
- link head_link: geometry visual mesh filename=package://hurobots/description_files/meshes/head_link.STL
- link left_ankle_pitch_link: geometry visual mesh filename=package://hurobots/description_files/meshes/left_ankle_pitc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
- link left_ankle_roll_link: geometry collision box size=0.20311 0.0647 0.01851; visual mesh filename=package://hurobots/description_files/meshes/left_ankle_roll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
- link left_elbow_link: geometry visual mesh filename=package://hurobots/description_files/meshes/left_elbow_link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
- link left_hip_pitch_link: geometry visual mesh filename=package://hurobots/description_files/meshes/left_hip_pitch_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
- link left_hip_roll_link: geometry visual mesh filename=package://hurobots/description_files/meshes/left_hip_roll_l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
- link left_hip_yaw_link: geometry visual mesh filename=package://hurobots/description_files/meshes/left_hip_yaw_li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
- link left_knee_link: geometry visual mesh filename=package://hurobots/description_files/meshes/left_knee_link.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
- link left_shoulder_pitch_link: geometry visual mesh filename=package://hurobots/description_files/meshes/left_shoulder_p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
- link left_shoulder_roll_link: geometry visual mesh filename=package://hurobots/description_files/meshes/left_shoulder_r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
- link left_shoulder_yaw_link: geometry collision sphere radius=0.04; visual mesh filename=package://hurobots/description_files/meshes/left_shoulder_y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
- link left_wrist_roll_rubber_hand: geometry collision mesh filename=package://hurobots/description_files/meshes/left_wrist_roll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; visual mesh filename=package://hurobots/description_files/meshes/left_wrist_roll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
- link logo_link: geometry visual mesh filename=package://hurobots/description_files/meshes/logo_link.STL
- link pelvis: geometry visual mesh filename=package://hurobots/description_files/meshes/pelvis.STL
- link pelvis_contour_link: geometry visual mesh filename=package://hurobots/description_files/meshes/pelvis_contour_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
- link right_ankle_pitch_link: geometry visual mesh filename=package://hurobots/description_files/meshes/right_ankle_pit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
- link right_ankle_roll_link: geometry collision box size=0.20311 0.0647 0.01851; visual mesh filename=package://hurobots/description_files/meshes/right_ankle_rol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
- link right_elbow_link: geometry visual mesh filename=package://hurobots/description_files/meshes/right_elbow_lin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
- link right_hip_pitch_link: geometry visual mesh filename=package://hurobots/description_files/meshes/right_hip_pitch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
- link right_hip_roll_link: geometry visual mesh filename=package://hurobots/description_files/meshes/right_hip_roll_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
- link right_hip_yaw_link: geometry visual mesh filename=package://hurobots/description_files/meshes/right_hip_yaw_l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
- link right_knee_link: geometry visual mesh filename=package://hurobots/description_files/meshes/right_knee_link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
- link right_shoulder_pitch_link: geometry visual mesh filename=package://hurobots/description_files/meshes/right_shoulder_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
- link right_shoulder_roll_link: geometry visual mesh filename=package://hurobots/description_files/meshes/right_shoulder_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
- link right_shoulder_yaw_link: geometry collision sphere radius=0.04; visual mesh filename=package://hurobots/description_files/meshes/right_shoulder_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
- link right_wrist_roll_rubber_hand: geometry collision mesh filename=package://hurobots/description_files/meshes/right_wrist_rol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; visual mesh filename=package://hurobots/description_files/meshes/right_wrist_rol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
- link torso_link: geometry collision mesh filename=package://hurobots/description_files/meshes/torso_link_23do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; visual mesh filename=package://hurobots/description_files/meshes/torso_link_23do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

File: description_files/urdf/g1_23dof_rubber_hands_only_palm_coll.urdf (robot description, URDF)
Before this commit: robot g1_23dof_rubber_hands, 31 links, 30 joints
Links:
- link head_link: geometry visual mesh filename=package://hurobots/description_files/meshes/head_link.STL
- link left_ankle_pitch_link: geometry visual mesh filename=package://hurobots/description_files/meshes/left_ankle_pitc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
- link left_ankle_roll_link: geometry collision box size=0.20311 0.0647 0.01851; visual mesh filename=package://hurobots/description_files/meshes/left_ankle_roll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
- link left_elbow_link: geometry visual mesh filename=package://hurobots/description_files/meshes/left_elbow_link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
- link left_hip_pitch_link: geometry visual mesh filename=package://hurobots/description_files/meshes/left_hip_pitch_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
- link left_hip_roll_link: geometry visual mesh filename=package://hurobots/description_files/meshes/left_hip_roll_l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
- link left_hip_yaw_link: geometry visual mesh filename=package://hurobots/description_files/meshes/left_hip_yaw_li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
- link left_knee_link: geometry visual mesh filename=package://hurobots/description_files/meshes/left_knee_link.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
- link left_shoulder_pitch_link: geometry visual mesh filename=package://hurobots/description_files/meshes/left_shoulder_p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
- link left_shoulder_roll_link: geometry visual mesh filename=package://hurobots/description_files/meshes/left_shoulder_r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
- link left_shoulder_yaw_link: geometry collision sphere radius=0.04; visual mesh filename=package://hurobots/description_files/meshes/left_shoulder_y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
- link left_wrist_roll_rubber_hand: geometry collision mesh filename=package://hurobots/description_files/meshes/left_rubber_pal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; collision mesh filename=package://hurobots/description_files/meshes/left_wrist_roll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
- link logo_link: geometry visual mesh filename=package://hurobots/description_files/meshes/logo_link.STL
- link pelvis: geometry visual mesh filename=package://hurobots/description_files/meshes/pelvis.STL
- link pelvis_contour_link: geometry visual mesh filename=package://hurobots/description_files/meshes/pelvis_contour_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
- link right_ankle_pitch_link: geometry visual mesh filename=package://hurobots/description_files/meshes/right_ankle_pit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
- link right_ankle_roll_link: geometry collision box size=0.20311 0.0647 0.01851; visual mesh filename=package://hurobots/description_files/meshes/right_ankle_rol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
- link right_elbow_link: geometry visual mesh filename=package://hurobots/description_files/meshes/right_elbow_lin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
- link right_hip_pitch_link: geometry visual mesh filename=package://hurobots/description_files/meshes/right_hip_pitch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
- link right_hip_roll_link: geometry visual mesh filename=package://hurobots/description_files/meshes/right_hip_roll_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
- link right_hip_yaw_link: geometry visual mesh filename=package://hurobots/description_files/meshes/right_hip_yaw_l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
- link right_knee_link: geometry visual mesh filename=package://hurobots/description_files/meshes/right_knee_link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
- link right_shoulder_pitch_link: geometry visual mesh filename=package://hurobots/description_files/meshes/right_shoulder_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
- link right_shoulder_roll_link: geometry visual mesh filename=package://hurobots/description_files/meshes/right_shoulder_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
- link right_shoulder_yaw_link: geometry collision sphere radius=0.04; visual mesh filename=package://hurobots/description_files/meshes/right_shoulder_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
- link right_wrist_roll_rubber_hand: geometry collision mesh filename=package://hurobots/description_files/meshes/right_rubber_pa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; collision mesh filename=package://hurobots/description_files/meshes/right_wrist_rol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
- link torso_link: geometry collision mesh filename=package://hurobots/description_files/meshes/torso_link_23do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; visual mesh filename=package://hurobots/description_files/meshes/torso_link_23do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

File: description_files/urdf/g1_29dof.urdf (robot description, URDF)
Before this commit: robot g1_29dof_rev_1_0, 56 links, 55 joints
Links:
- link head_link: geometry collision mesh filename=package://hurobots/description_files/meshes/head_link.STL; visual mesh filename=package://hurobots/description_files/meshes/head_link.STL
- link left_ankle_pitch_link: geometry collision mesh filename=package://hurobots/description_files/meshes/left_ankle_pitc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; visual mesh filename=package://hurobots/description_files/meshes/left_ankle_pitc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
- link left_ankle_roll_link: geometry collision sphere radius=0.005; collision sphere radius=0.005
- link left_elbow_link: geometry collision mesh filename=package://hurobots/description_files/meshes/left_elbow_link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; visual mesh filename=package://hurobots/description_files/meshes/left_elbow_link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
- link left_hip_pitch_link: geometry collision mesh filename=package://hurobots/description_files/meshes/left_hip_pitch_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; visual mesh filename=package://hurobots/description_files/meshes/left_hip_pitch_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
- link left_hip_roll_link: geometry collision mesh filename=package://hurobots/description_files/meshes/left_hip_roll_l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; visual mesh filename=package://hurobots/description_files/meshes/left_hip_roll_l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
- link left_hip_yaw_link: geometry collision mesh filename=package://hurobots/description_files/meshes/left_hip_yaw_li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; visual mesh filename=package://hurobots/description_files/meshes/left_hip_yaw_li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
- link left_knee_link: geometry collision mesh filename=package://hurobots/description_files/meshes/left_knee_link.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; visual mesh filename=package://hurobots/description_files/meshes/left_knee_link.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
- link left_rubber_hand: geometry visual mesh filename=package://hurobots/description_files/meshes/left_rubber_han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
- link left_shoulder_pitch_link: geometry collision cylinder length=0.05 radius=0.03; visual mesh filename=package://hurobots/description_files/meshes/left_shoulder_p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
- link left_shoulder_roll_link: geometry collision cylinder length=0.03 radius=0.03; visual mesh filename=package://hurobots/description_files/meshes/left_shoulder_r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
- link left_shoulder_yaw_link: geometry collision mesh filename=package://hurobots/description_files/meshes/left_shoulder_y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; visual mesh filename=package://hurobots/description_files/meshes/left_shoulder_y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
- link left_wrist_pitch_link: geometry collision mesh filename=package://hurobots/description_files/meshes/left_wrist_pitc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; visual mesh filename=package://hurobots/description_files/meshes/left_wrist_pitc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
- link left_wrist_roll_link: geometry collision mesh filename=package://hurobots/description_files/meshes/left_wrist_roll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; visual mesh filename=package://hurobots/description_files/meshes/left_wrist_roll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
- link left_wrist_yaw_link: geometry collision mesh filename=package://hurobots/description_files/meshes/left_wrist_yaw_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; visual mesh filename=package://hurobots/description_files/meshes/left_wrist_yaw_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
- link logo_link: geometry collision mesh filename=package://hurobots/description_files/meshes/logo_link.STL; visual mesh filename=package://hurobots/description_files/meshes/logo_link.STL
- link pelvis: geometry visual mesh filename=package://hurobots/description_files/meshes/pelvis.STL
- link pelvis_contour_link: geometry collision mesh filename=package://hurobots/description_files/meshes/pelvis_contour_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; visual mesh filename=package://hurobots/description_files/meshes/pelvis_contour_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
- link right_ankle_pitch_link: geometry collision mesh filename=package://hurobots/description_files/meshes/right_ankle_pit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; visual mesh filename=package://hurobots/description_files/meshes/right_ankle_pit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
- link right_ankle_roll_link: geometry collision sphere radius=0.005; collision sphere radius=0.005
- link right_elbow_link: geometry collision mesh filename=package://hurobots/description_files/meshes/right_elbow_lin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; visual mesh filename=package://hurobots/description_files/meshes/right_elbow_lin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
- link right_hip_pitch_link: geometry collision mesh filename=package://hurobots/description_files/meshes/right_hip_pitch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; visual mesh filename=package://hurobots/description_files/meshes/right_hip_pitch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
- link right_hip_roll_link: geometry collision mesh filename=package://hurobots/description_files/meshes/right_hip_roll_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; visual mesh filename=package://hurobots/description_files/meshes/right_hip_roll_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
- link right_hip_yaw_link: geometry collision mesh filename=package://hurobots/description_files/meshes/right_hip_yaw_l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; visual mesh filename=package://hurobots/description_files/meshes/right_hip_yaw_l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
- link right_knee_link: geometry collision mesh filename=package://hurobots/description_files/meshes/right_knee_link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; visual mesh filename=package://hurobots/description_files/meshes/right_knee_link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
- link right_rubber_hand: geometry visual mesh filename=package://hurobots/description_files/meshes/right_rubber_ha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
- link right_shoulder_pitch_link: geometry collision cylinder length=0.05 radius=0.03; visual mesh filename=package://hurobots/description_files/meshes/right_shoulder_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
- link right_shoulder_roll_link: geometry collision cylinder length=0.03 radius=0.03; visual mesh filename=package://hurobots/description_files/meshes/right_shoulder_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
- link right_shoulder_yaw_link: geometry collision mesh filename=package://hurobots/description_files/meshes/right_shoulder_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; visual mesh filename=package://hurobots/description_files/meshes/right_shoulder_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
- link right_wrist_pitch_link: geometry collision mesh filename=package://hurobots/description_files/meshes/right_wrist_pit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; visual mesh filename=package://hurobots/description_files/meshes/right_wrist_pit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
- link right_wrist_roll_link: geometry collision mesh filename=package://hurobots/description_files/meshes/right_wrist_rol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; visual mesh filename=package://hurobots/description_files/meshes/right_wrist_rol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
- link right_wrist_yaw_link: geometry collision mesh filename=package://hurobots/description_files/meshes/right_wrist_yaw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; visual mesh filename=package://hurobots/description_files/meshes/right_wrist_yaw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
- link torso_link: geometry collision mesh filename=package://hurobots/description_files/meshes/torso_link_rev_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; visual mesh filename=package://hurobots/description_files/meshes/torso_link_rev_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
- link waist_roll_link: geometry visual mesh filename=package://hurobots/description_files/meshes/waist_roll_link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
- link waist_yaw_link: geometry visual mesh filename=package://hurobots/description_files/meshes/waist_yaw_link_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
