Commit message: Add lidar visualization for g1

File: description_files/urdf/g1_29dof.urdf (robot description, URDF)
Before this commit: robot g1_29dof_rev_1_0, 56 links, 55 joints
Links:
- added link livox_frame
Joints:
- added joint livox_joint: type fixed, parent mid360_link, child livox_frame, origin xyz=0.0 0.0 0.0 rpy=3.141561 0 0
